File: DehneEVSE.sch (KiCad schematic (older format))
At the start: 46 parts, among them J1 Connector1, J3 FC68131, J4 FC68131, J5 FC68131, K1 G5NB-1A Relay 5VDC, Q1 PN2222A, T1 VB_05-1-12, T2 VB_05-1-12, T3 VB_05-1-12, U1 Arduino Nano 33 IoT, U2 IRM-05-5, U3 LT1498IN8#PBF, U4 mcp6291-e_p-nd, U5 mcp6291-e_p-nd, U6 mcp6291-e_p-nd

Commit message: renamed to DehneEVSE
Parts:
- removed U3: LT1498IN8#PBF, Package_DIP:DIP-8_W7.62mm, symbol EVChargingStationParts:LF353P
- added U3: LT1498IN8, Package_DIP:DIP-8_W7.62mm, symbol DehneEVSESymbols:LT1498IN8
- J1: footprint EVChargingStation:conn_08x02_wago -> DehneEVSEFootPrints:conn_08x02_wago; symbol EVChargingStationParts:Connector1 -> DehneEVSESymbols:Connector1
- J3, J4, J5: footprint EVChargingStation:CLIFF_FC68131 -> DehneEVSEFootPrints:CLIFF_FC68131; symbol EVChargingStationParts:FC68131 -> DehneEVSESymbols:FC68131
- K1: footprint EVChargingStation:Omron-GSNB-1A -> DehneEVSEFootPrints:Omron-GSNB-1A; symbol EVChargingStationParts:Relay_NO -> DehneEVSESymbols:Relay_NO
- T1, T2, T3: footprint EVChargingStation:VB_05-1-12 -> DehneEVSEFootPrints:VB_05-1-12; symbol EVChargingStationParts:VB_05-1-12 -> DehneEVSESymbols:VB_05-1-12
- U1: footprint EVChargingStation:Arduino Nano - THT -> DehneEVSEFootPrints:Arduino Nano - THT; symbol EVChargingStationParts:ABX00027 -> DehneEVSESymbols:ABX00027
- U2: footprint EVChargingStation:CONV_IRM-05-5 -> DehneEVSEFootPrints:CONV_IRM-05-5; symbol EVChargingStationParts:IRM-05-5 -> DehneEVSESymbols:IRM-05-5
- U4, U5, U6: symbol EVChargingStationParts:mcp6291-e_p-nd -> DehneEVSESymbols:mcp6291-e_p-nd
Connections:
- net +12VDC: now also U3.8 (V+)
- net -12VDC: now also U3.4 (V-)
- net GND: now also U3.5 (+)
- net PWM: now also U3.3 (+)
- net at R4.2, R5.1: now also U3.2 (-)
- net at R6.2: now also U3.1 (OUT)
- new net: U3.6 (-), U3.7 (OUT)
Changed lines of the file:
@@
 $EndDescr
 $Comp
-L EVChargingStationParts:IRM-05-5 U2
+L DehneEVSESymbols:IRM-05-5 U2
 U 1 1 6032F4DA
 P 4750 1900
 F 0 "U2" H 4750 2367 50  0000 C CNN
 F 1 "IRM-05-5" H 4750 2276 50  0000 C CNN
-F 2 "EVChargingStation:CONV_IRM-05-5" H 4750 1900 50  0001 L BNN
+F 2 "DehneEVSEFootPrints:CONV_IRM-05-5" H 4750 1900 50  0001 L BNN
 F 3 "" H 4750 1900 50  0001 L BNN
 F 4 "None" H 4750 1900 50  0001 L BNN "PRICE"
@@
 $EndComp
 $Comp
-L EVChargingStationParts:Relay_NO K1
+L DehneEVSESymbols:Relay_NO K1
 U 1 1 6034E03E
 P 7650 4500
 F 0 "K1" V 7450 4800 60  0000 R CNN
 F 1 "G5NB-1A Relay 5VDC" V 8000 5650 60  0000 R CNN
-F 2 "EVChargingStation:Omron-GSNB-1A" H 7650 4500 60  0001 C CNN
+F 2 "DehneEVSEFootPrints:Omron-GSNB-1A" H 7650 4500 60  0001 C CNN
 F 3 "" H 7650 4500 60  0000 C CNN
 	1    7650 4500
@@
 	1950 2350 1800 2350
 $Comp
-L EVChargingStationParts:VB_05-1-12 T1
+L DehneEVSESymbols:VB_05-1-12 T1
 U 1 1 60521BCF
 P 2300 6300
 F 0 "T1" H 2050 6550 50  0000 C CNN
 F 1 "VB_05-1-12" H 2250 6050 50  0000 C CNN
-F 2 "EVChargingStation:VB_05-1-12" H 2200 6300 50  0001 C CNN
+F 2 "DehneEVSEFootPrints:VB_05-1-12" H 2200 6300 50  0001 C CNN
 F 3 "" H 2200 6300 50  0001 C CNN
 	1    2300 6300
@@
 VOLTAGE_SENS_L3_READ
 $Comp
-L EVChargingStationParts:FC68131 J3
+L DehneEVSESymbols:FC68131 J3
 U 1 1 606C7A4E
 P 1450 3150
 F 0 "J3" H 1494 3331 50  0000 C CNN
 F 1 "FC68131" H 1494 3240 50  0000 C CNN
-F 2 "EVChargingStation:CLIFF_FC68131" H 1450 3150 50  0001 L BNN
+F 2 "DehneEVSEFootPrints:CLIFF_FC68131" H 1450 3150 50  0001 L BNN
 F 3 "" H 1450 3150 50  0001 L BNN
 F 4 "6.00 mm" H 1450 3150 50  0001 L BNN "MAXIMUM_PACKAGE_HEIGHT"
@@
 $EndComp
 $Comp
-L EVChargingStationParts:FC68131 J4
+L DehneEVSESymbols:FC68131 J4
 U 1 1 606C8ED9
 P 1450 3650
 F 0 "J4" H 1494 3831 50  0000 C CNN
 F 1 "FC68131" H 1494 3740 50  0000 C CNN
-F 2 "EVChargingStation:CLIFF_FC68131" H 1450 3650 50  0001 L BNN
+F 2 "DehneEVSEFootPrints:CLIFF_FC68131" H 1450 3650 50  0001 L BNN
 F 3 "" H 1450 3650 50  0001 L BNN
 F 4 "6.00 mm" H 1450 3650 50  0001 L BNN "MAXIMUM_PACKAGE_HEIGHT"
@@
 $EndComp
 $Comp
-L EVChargingStationParts:FC68131 J5
+L DehneEVSESymbols:FC68131 J5
 U 1 1 606C9CAA
 P 1450 4150
 F 0 "J5" H 1494 4331 50  0000 C CNN
 F 1 "FC68131" H 1494 4240 50  0000 C CNN
-F 2 "EVChargingStation:CLIFF_FC68131" H 1450 4150 50  0001 L BNN
+F 2 "DehneEVSEFootPrints:CLIFF_FC68131" H 1450 4150 50  0001 L BNN
 F 3 "" H 1450 4150 50  0001 L BNN
 F 4 "6.00 mm" H 1450 4150 50  0001 L BNN "MAXIMUM_PACKAGE_HEIGHT"
@@
 Connection ~ 7250 2250
 $Comp
-L EVChargingStationParts:ABX00027 U1
+L DehneEVSESymbols:ABX00027 U1
 U 1 1 603AB8EE
 P 4750 3800
 F 0 "U1" H 4750 4967 50  0000 C CNN
 F 1 "Arduino Nano 33 IoT" H 4750 4876 50  0000 C CNN
-F 2 "EVChargingStation:Arduino Nano - THT" H 2700 4650 50  0001 L BNN
+F 2 "DehneEVSEFootPrints:Arduino Nano - THT" H 2700 4650 50  0001 L BNN
 F 3 "" H 4750 3800 50  0001 L BNN
 F 4 "ATSAMD21G18A Arduino Nano 33 IoT SAM D ARM® Cortex®-M0+ MCU 32-Bit Embedded Evaluation Board" H 2650 2600 50  0001 L BNN "DESCRIPTION"
@@
 Connection ~ 5550 4700
 $Comp
-L EVChargingStationParts:mcp6291-e_p-nd U4
+L DehneEVSESymbols:mcp6291-e_p-nd U4
 U 1 1 6047606D
 P 2600 8650
@@
 	8800 2100 8800 2200
 $Comp
-L EVChargingStationParts:LF353P U3
-U 1 1 605C9FC7
-P 10750 1900
-F 0 "U3" H 10750 2100 50  0000 L CNN
-F 1 "LT1498IN8#PBF" H 10550 1650 50  0000 L CNN
-F 2 "Package_DIP:DIP-8_W7.62mm" H 10750 1900 50  0001 C CNN
-F 3 "https://www.ti.com/lit/ds/slos012c/slos012c.pdf?ts=1615223850164" H 10750 1900 50  0001 C CNN
-	1    10750 1900
-	1    0    0    -1
-$EndComp
-$Comp
-L EVChargingStationParts:Connector1 J1
+L DehneEVSESymbols:Connector1 J1
 U 1 1 6077AEE9
 P 1500 2100
 F 0 "J1" H 1533 2675 50  0000 C CNN
 F 1 "Connector1" H 1533 2584 50  0000 C CNN
-F 2 "EVChargingStation:conn_08x02_wago" H 2000 2150 50  0001 C CNN
+F 2 "DehneEVSEFootPrints:conn_08x02_wago" H 2000 2150 50  0001 C CNN
 F 3 "" H 2000 2150 50  0001 C CNN
 	1    1500 2100
@@
 Text GLabel 8600 2500 3    50   Input ~ 0
 -12VDC
-$Comp
-L EVChargingStationParts:LF353P U3
-U 2 1 60422890
-P 10800 3050
-F 0 "U3" H 10850 3250 50  0000 C CNN
-F 1 "LT1498IN8#PBF" H 10850 2800 50  0000 C CNN
-F 2 "Package_DIP:DIP-8_W7.62mm" H 10800 3050 50  0001 C CNN
-F 3 "https://www.ti.com/lit/ds/slos012c/slos012c.pdf?ts=1615223850164" H 10800 3050 50  0001 C CNN
-	2    10800 3050
-	1    0    0    -1
-$EndComp
 Wire Wire Line
 	10450 1800 10400 1800
@@
 Wire Wire Line
 	10300 2950 10300 3000
-$Comp
-L EVChargingStationParts:LF353P U3
-U 3 1 60523284
-P 9400 2100
-F 0 "U3" H 9400 2300 50  0000 L CNN
-F 1 "LT1498IN8#PBF" H 9400 1950 50  0000 L CNN
-F 2 "Package_DIP:DIP-8_W7.62mm" H 9400 2100 50  0001 C CNN
-F 3 "https://www.ti.com/lit/ds/slos012c/slos012c.pdf?ts=1615223850164" H 9400 2100 50  0001 C CNN
-	3    9400 2100
-	1    0    0    -1
-$EndComp
 Text GLabel 5600 3100 2    50   Input ~ 0
 +3V3
@@
 	2500 8350 2500 8200
 $Comp
-L EVChargingStationParts:VB_05-1-12 T2
+L DehneEVSESymbols:VB_05-1-12 T2
 U 1 1 6083B3E5
 P 5350 6300
 F 0 "T2" H 5100 6550 50  0000 C CNN
 F 1 "VB_05-1-12" H 5300 6050 50  0000 C CNN
-F 2 "EVChargingStation:VB_05-1-12" H 5250 6300 50  0001 C CNN
+F 2 "DehneEVSEFootPrints:VB_05-1-12" H 5250 6300 50  0001 C CNN
 F 3 "" H 5250 6300 50  0001 C CNN
 	1    5350 6300
@@
 	6200 6700 6200 6750
 $Comp
-L EVChargingStationParts:VB_05-1-12 T3
+L DehneEVSESymbols:VB_05-1-12 T3
 U 1 1 608499D2
 P 8400 6300
 F 0 "T3" H 8150 6550 50  0000 C CNN
 F 1 "VB_05-1-12" H 8350 6050 50  0000 C CNN
-F 2 "EVChargingStation:VB_05-1-12" H 8300 6300 50  0001 C CNN
+F 2 "DehneEVSEFootPrints:VB_05-1-12" H 8300 6300 50  0001 C CNN
 F 3 "" H 8300 6300 50  0001 C CNN
 	1    8400 6300
@@
 	5550 8650 5600 8650
 $Comp
-L EVChargingStationParts:mcp6291-e_p-nd U5
+L DehneEVSESymbols:mcp6291-e_p-nd U5
 U 1 1 608C29C3
 P 5250 8650
@@
 	8250 8650 8300 8650
 $Comp
-L EVChargingStationParts:mcp6291-e_p-nd U6
+L DehneEVSESymbols:mcp6291-e_p-nd U6
 U 1 1 608D1798
 P 7950 8650
@@
 	-1   0    0    1
 $EndComp
+$Comp
+L DehneEVSESymbols:LT1498IN8 U3
+U 1 1 604B399B
+P 10750 1900
+F 0 "U3" H 10750 2267 50  0000 C CNN
+F 1 "LT1498IN8" H 10750 2176 50  0000 C CNN
+F 2 "Package_DIP:DIP-8_W7.62mm" H 10750 1900 50  0001 C CNN
+F 3 "https://www.analog.com/media/en/technical-documentation/data-sheets/14989fg.pdf" H 10750 1900 50  0001 C CNN
+	1    10750 1900
+	1    0    0    -1
+$EndComp
+$Comp
+L DehneEVSESymbols:LT1498IN8 U3
+U 2 1 604B4851
+P 10800 3050
+F 0 "U3" H 10800 3417 50  0000 C CNN
+F 1 "LT1498IN8" H 10800 3326 50  0000 C CNN
+F 2 "Package_DIP:DIP-8_W7.62mm" H 10800 3050 50  0001 C CNN
+F 3 "https://www.analog.com/media/en/technical-documentation/data-sheets/14989fg.pdf" H 10800 3050 50  0001 C CNN
+	2    10800 3050
+	1    0    0    -1
+$EndComp
+$Comp
+L DehneEVSESymbols:LT1498IN8 U3
+U 3 1 604B5141
+P 9400 2100
+F 0 "U3" H 9630 2146 50  0000 L CNN
+F 1 "LT1498IN8" H 9630 2055 50  0000 L CNN
+F 2 "Package_DIP:DIP-8_W7.62mm" H 9400 2100 50  0001 C CNN
+F 3 "https://www.analog.com/media/en/technical-documentation/data-sheets/14989fg.pdf" H 9400 2100 50  0001 C CNN
+	3    9400 2100
+	1    0    0    -1
+$EndComp
 $EndSCHEMATC

Commit message: minor updates
Parts:
- U2: value IRM-05-5 -> NMA0512SC
Changed lines of the file:
@@
 P 4750 1900
 F 0 "U2" H 4750 2367 50  0000 C CNN
-F 1 "IRM-05-5" H 4750 2276 50  0000 C CNN
+F 1 "NMA0512SC" H 4750 2276 50  0000 C CNN
 F 2 "DehneEVSEFootPrints:CONV_IRM-05-5" H 4750 1900 50  0001 L BNN
 F 3 "" H 4750 1900 50  0001 L BNN

Commit message: rev 1.4
Parts:
- removed U4, U5, U6: mcp6291-e_p-nd, Package_DIP:DIP-8_W7.62mm, symbol DehneEVSESymbols:mcp6291-e_p-nd
- added U4, U5, U6: MCP602T, Package_SO:SOIC-8_3.9x4.9mm_P1.27mm, symbol DehneEVSESymbols:MCP602T
- Q1: footprint Package_TO_SOT_THT:TO-92_Inline -> Package_TO_SOT_THT:TO-92_Inline_Wide
- R10, R12, R14: value 100k -> 10k
- R13, R17, R9: value 10k -> 100k
- U1: footprint DehneEVSEFootPrints:Arduino Nano - THT -> DehneEVSEFootPrints:Arduino_Nano_33_iot__SMT
Connections:
- net +3V3: now also U4.8 (V+), U5.8 (V+), U6.8 (V+)
- net CURRENT_SENS_L1_READ: now also R12.2, U4.7 (out); no longer R16.2
- net CURRENT_SENS_L2_READ: now also R16.2, U5.7 (out); no longer R18.2
- net CURRENT_SENS_L3_READ: now also U6.7 (out)
- net CUR_SENS_L1: now also U4.5 (+)
- net CUR_SENS_L2: now also U5.5 (+)
- net CUR_SENS_L3: now also U6.5 (+)
- net GND: now also R10.2, R11.1, R14.2, R18.2, U4.4 (V-), U5.4 (V-), U6.4 (V-); no longer R11.2, R13.2, R17.1, R9.2
- net MAINS_L1: no longer K1.2
- net MAINS_N: now also K1.2
- net VOLTAGE_SENS_L1_READ: now also U4.1 (out), U4.2 (-); no longer R10.2, R9.1
- net VOLTAGE_SENS_L2_READ: now also U5.1 (out), U5.2 (-); no longer R11.1, R12.2
- net VOLTAGE_SENS_L3_READ: now also U6.1 (out), U6.2 (-); no longer R13.1, R14.2
- net at R15.2, R16.1: now also U5.6 (-)
- net at R10.1: now also R9.2, U4.3 (+); no longer D1.1 (K)
- net at R12.1: now also R11.2, U4.6 (-); no longer D4.1 (K)
- net at R14.1: now also R13.2, U5.3 (+); no longer D5.1 (K)
- net at R17.2, R18.1: now also U6.3 (+)
- net at R19.2, R20.1: now also U6.6 (-)
- new net: D1.1 (K), R9.1
- new net: D4.1 (K), R13.1
- new net: D5.1 (K), R17.1
Other:
- note added: "1x gain buffer to overcome\n4k7 pull-up at A4 & A5"
- note added: "AC 50Hz\nVpp -1.4/-1.4V"
- note added: "AC 50Hz\nVpp -28/28V"
- note added: "Voltage and current sensing - Phase1"
- note added: "Voltage and current sensing - Phase2"
- note added: "Voltage and current sensing - Phase3"
- note added: "only positive wave\n2x gain: 1.4 to 2.8V"
- note removed: "Charging load / current sensing L1, L2 & L3"
- note removed: "Mains Voltage sensing L1, L2 & L3"
