File: DehneEVSE.kicad_pcb (KiCad board)
At the start: 2 copper layers, 188 x 98 mm, 57 parts, among them J1 Connector1, J3 FC68131, J4 FC68131, J5 FC68131, K1 G5NB-1A Relay 5VDC, Q1 PN2222A, T1 VB_05-1-12, T2 VB_05-1-12, T3 VB_05-1-12, U1 Arduino Nano 33 IoT, U2 IRM-05-5, U3 LT1498IN8, U4 mcp6291-e_p-nd, U5 mcp6291-e_p-nd, U6 mcp6291-e_p-nd

Commit message: rev 1.4
Parts:
- Q1: footprint Package_TO_SOT_THT:TO-92_Inline -> Package_TO_SOT_THT:TO-92_Inline_Wide
- R10, R12, R14: value 100k -> 10k
- R13, R17, R9: value 10k -> 100k
- U1: footprint DehneEVSEFootPrints:Arduino Nano - THT -> DehneEVSEFootPrints:Arduino_Nano_33_iot__SMT
- U2: value IRM-05-5 -> NMA0512SC
- U4, U5, U6: value mcp6291-e_p-nd -> MCP602T; footprint Package_DIP:DIP-8_W7.62mm -> Package_SO:SOIC-8_3.9x4.9mm_P1.27mm
- moved REF** 140.2 mm to (137.5, 134.8)
- moved U6 116.6 mm to (170.8, 124.5)
- moved R19 116.0 mm to (165.8, 134.0), turned to 0 degrees
- moved U1 115.4 mm to (266.8, 130.0), turned to 0 degrees
- moved R20 112.9 mm to (176.0, 130.8), turned to 180 degrees
- moved REF** 107.5 mm to (152.8, 135.2)
- moved R18 107.3 mm to (165.8, 137.2), turned to 0 degrees
- moved R1 101.8 mm to (282.2, 148.3), turned to 270 degrees
- moved R7 96.6 mm to (275.4, 148.2), turned to 270 degrees
- moved R17 91.2 mm to (175.8, 140.5), turned to 180 degrees
- moved R2 90.4 mm to (278.8, 158.5), turned to 90 degrees
- moved D6 86.9 mm to (269.0, 157.5), turned to 90 degrees
- moved R8 86.2 mm to (272.0, 158.5), turned to 90 degrees
- moved U5 83.1 mm to (195.2, 124.5)
- moved R16 67.0 mm to (200.2, 130.5), turned to 180 degrees
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Connections:
- K1 pad 2: MAINS_L1 -> MAINS_N
- R10 pad 1: Net-(D1-Pad1) -> Net-(R10-Pad1)
- R10 pad 2: VOLTAGE_SENS_L1_READ -> GND
- R11 pad 1: VOLTAGE_SENS_L2_READ -> GND
- R11 pad 2: GND -> Net-(R11-Pad2)
- R12 pad 1: Net-(D4-Pad1) -> Net-(R11-Pad2)
- R12 pad 2: VOLTAGE_SENS_L2_READ -> CURRENT_SENS_L1_READ
- R13 pad 1: VOLTAGE_SENS_L3_READ -> Net-(D4-Pad1)
- R13 pad 2: GND -> Net-(R13-Pad2)
- R14 pad 1: Net-(D5-Pad1) -> Net-(R13-Pad2)
- R14 pad 2: VOLTAGE_SENS_L3_READ -> GND
- R16 pad 2: CURRENT_SENS_L1_READ -> CURRENT_SENS_L2_READ
- R17 pad 1: GND -> Net-(D5-Pad1)
- R18 pad 2: CURRENT_SENS_L2_READ -> GND
- R9 pad 1: VOLTAGE_SENS_L1_READ -> Net-(D1-Pad1)
- R9 pad 2: GND -> Net-(R10-Pad1)
- U4 pad 1: (no net) -> VOLTAGE_SENS_L1_READ
- U4 pad 2: Net-(R15-Pad2) -> VOLTAGE_SENS_L1_READ
- U4 pad 3: CUR_SENS_L1 -> Net-(R10-Pad1)
- U4 pad 4: +3V3 -> GND
- U4 pad 5: (no net) -> CUR_SENS_L1
- U4 pad 6: CURRENT_SENS_L1_READ -> Net-(R11-Pad2)
- U4 pad 7: GND -> CURRENT_SENS_L1_READ
- U4 pad 8: (no net) -> +3V3
- U5 pad 1: (no net) -> VOLTAGE_SENS_L2_READ
- U5 pad 2: Net-(R17-Pad2) -> VOLTAGE_SENS_L2_READ
- U5 pad 3: CUR_SENS_L2 -> Net-(R13-Pad2)
- U5 pad 4: +3V3 -> GND
- U5 pad 5: (no net) -> CUR_SENS_L2
- U5 pad 6: CURRENT_SENS_L2_READ -> Net-(R15-Pad2)
- U5 pad 7: GND -> CURRENT_SENS_L2_READ
- U5 pad 8: (no net) -> +3V3
- U6 pad 1: (no net) -> VOLTAGE_SENS_L3_READ
- U6 pad 2: Net-(R19-Pad2) -> VOLTAGE_SENS_L3_READ
- U6 pad 3: CUR_SENS_L3 -> Net-(R17-Pad2)
- U6 pad 4: +3V3 -> GND
- U6 pad 5: (no net) -> CUR_SENS_L3
- U6 pad 6: CURRENT_SENS_L3_READ -> Net-(R19-Pad2)
- U6 pad 7: GND -> CURRENT_SENS_L3_READ
- U6 pad 8: (no net) -> +3V3
Routing:
- net CUR_SENS_L3: track 11.5 -> 167.1 mm, vias 0 -> 2
- net CUR_SENS_L2: track 12.0 -> 125.0 mm, vias 0 -> 2
- net CURRENT_SENS_L3_READ: track 204.0 -> 111.6 mm, vias 0 -> 2
- net CURRENT_SENS_L2_READ: track 170.6 -> 84.4 mm, vias 0 -> 2
- net CURRENT_SENS_L1_READ: track 135.8 -> 57.9 mm, vias 0 -> 2
- net CUR_SENS_L1: track 11.8 -> 85.7 mm, vias 0 -> 2
- net +5V: track 249.5 -> 321.7 mm
- net VOLTAGE_SENS_L3_READ: track 60.0 -> 124.9 mm, vias 1 -> 2
- net DC_RELAY: track 106.2 -> 53.2 mm, vias 0 -> 1
- net VOLTAGE_SENS_L2_READ: track 56.8 -> 96.5 mm, vias 1 -> 2
- net Net-(R6-Pad2): track 52.8 -> 15.4 mm, vias 2 -> 0
- net MAINS_L1: track 105.2 -> 77.3 mm
- net Net-(R10-Pad1): track 0.00 -> 22.6 mm
- net Net-(R13-Pad2): track 0.00 -> 22.1 mm
- net MAINS_N: track 148.1 -> 168.3 mm
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Other:
- board text added: "Current sens.L1"
- board text added: "Current sens.L2"
- board text added: "Current sens.L3"
- board text added: "dehnes.com - rev 1.4"
- board text removed: "C.sens.L1"
- board text removed: "C.sens.L2"
- board text removed: "C.sens.L3"
- board text removed: "dehnes.com - rev 1.3"

Commit message: rev 1.4
Routing:
- net VOLTAGE_SENS_L3_READ: track 124.9 -> 119.7 mm
- net VOLTAGE_SENS_L2_READ: track 96.5 -> 92.6 mm
